File: PeripheralSOM.kicad_pcb (KiCad board)
At the start: 4 copper layers, 53.5 x 37.8 mm, 121 parts, among them J1 SWD, J2 USB4215-03-A, J4 52465-2470, SW1 RST, SW2 BOOT, U1 STM32L431CBTx, U2 TPS5405DR, U3 LT1963AEST-3.3#TRPBF, U4 TCAN337, U5 CDSOT23-T24CAN, U6 TPS2115ADRBR, U7 LM76202QPWPRQ1, U8 CP2102N-A02-GQFN24, U9 74AHC1G32, Y1 8M

Commit message: laksee
Parts:
- removed JP2: EN, Jumper:SolderJumper-2_P1.3mm_Open_TrianglePad1.0x1.5mm
- added D15: 1N5819HW, Diode_SMD:D_SOD-123, F.Cu at (124.1, 107.8)
- moved C18 0.40 mm to (120.6, 106.2)
- moved D5 0.20 mm to (129.0, 107.8)
Other:
- board text added: "Peripheral SOM Rev B.1"
- board text removed: "Peripheral SOM Rev B"
